File: lopill.kicad/lopill.kicad_pcb (KiCad board)
At the start: 2 copper layers, 23 x 59.5 mm, 34 parts, among them J1 Pins Left, J2 SWD, J3 USB_B_Micro, J4 Pins Right, SW1 Reset, U1 XC6206PxxxMR, U2 STM32L052C8Tx, Y1 8MHz, Y2 32.768KHz

Commit message: Add JLCJLCJLCJLC placeholder
Other:
- board text added: "JLCJLCJLCJLC"
Changed lines of the file:
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@@
   (general
     (thickness 1.6)
-    (drawings 31)
+    (drawings 32)
     (tracks 572)
     (zones 0)
@@
     (32 B.Adhes user hide)
     (33 F.Adhes user hide)
-    (34 B.Paste user hide)
+    (34 B.Paste user)
     (35 F.Paste user hide)
     (36 B.SilkS user)
     (37 F.SilkS user)
     (38 B.Mask user)
-    (39 F.Mask user)
+    (39 F.Mask user hide)
     (40 Dwgs.User user hide)
     (41 Cmts.User user hide)
@@
     (45 Margin user hide)
     (46 B.CrtYd user)
-    (47 F.CrtYd user)
-    (48 B.Fab user hide)
+    (47 F.CrtYd user hide)
+    (48 B.Fab user)
     (49 F.Fab user hide)
   )
@@
       (rotate (xyz 0 0 0))
     )
+  )
+  (gr_text JLCJLCJLCJLC (at 60.8584 79.2988) (layer B.SilkS)
+    (effects (font (size 1 1) (thickness 0.15)) (justify mirror))
   )
   (gr_text "LoPill v1\nby spbnick" (at 60.96 47.625) (layer B.SilkS)
@@
   (segment (start 68.58 88.282522) (end 68.58 88.9) (width 0.5) (layer F.Cu) (net 30))
   (segment (start 67.280999 86.983521) (end 68.58 88.282522) (width 0.5) (layer F.Cu) (net 30))
-  (segment (start 67.37599 90.10401) (end 68.58 88.9) (width 0.5) (layer B.Cu) (net 30) (status 1000000))
-  (segment (start 62.26 88.98) (end 63.38401 90.10401) (width 0.5) (layer B.Cu) (net 30) (status 1000000))
+  (segment (start 67.37599 90.10401) (end 68.58 88.9) (width 0.5) (layer B.Cu) (net 30))
+  (segment (start 62.26 88.98) (end 63.38401 90.10401) (width 0.5) (layer B.Cu) (net 30))
   (segment (start 63.38401 90.10401) (end 67.37599 90.10401) (width 0.5) (layer B.Cu) (net 30))
   (segment (start 65.17558 61.973796) (end 65.900794 62.69901) (width 0.25) (layer F.Cu) (net 31))
@@
   (segment (start 69.754001 69.754001) (end 68.58 68.58) (width 0.25) (layer B.Cu) (net 31))
   (segment (start 69.754001 89.463521) (end 69.754001 69.754001) (width 0.25) (layer B.Cu) (net 31))
-  (segment (start 62.303166 90.223834) (end 62.757352 90.67802) (width 0.25) (layer B.Cu) (net 31) (status 1000000))
-  (segment (start 62.757352 90.67802) (end 68.539504 90.678018) (width 0.25) (layer B.Cu) (net 31) (status 1000000))
-  (segment (start 62.984001 89.542999) (end 62.303166 90.223834) (width 0.25) (layer F.Cu) (net 31) (status 1000000))
-  (via (at 62.303166 90.223834) (size 0.8) (drill 0.4) (layers F.Cu B.Cu) (net 31) (status 1000000))
-  (segment (start 61.61 87.98) (end 62.643202 87.98) (width 0.25) (layer F.Cu) (net 31) (status 1000000))
-  (segment (start 62.643202 87.98) (end 62.984001 88.320799) (width 0.25) (layer F.Cu) (net 31) (status 1000000))
-  (segment (start 62.984001 88.320799) (end 62.984001 89.542999) (width 0.25) (layer F.Cu) (net 31) (status 1000000))
+  (segment (start 62.303166 90.223834) (end 62.757352 90.67802) (width 0.25) (layer B.Cu) (net 31))
+  (segment (start 62.757352 90.67802) (end 68.539504 90.678018) (width 0.25) (layer B.Cu) (net 31))
+  (segment (start 62.984001 89.542999) (end 62.303166 90.223834) (width 0.25) (layer F.Cu) (net 31))
+  (via (at 62.303166 90.223834) (size 0.8) (drill 0.4) (layers F.Cu B.Cu) (net 31))
+  (segment (start 61.61 87.98) (end 62.643202 87.98) (width 0.25) (layer F.Cu) (net 31))
+  (segment (start 62.643202 87.98) (end 62.984001 88.320799) (width 0.25) (layer F.Cu) (net 31))
+  (segment (start 62.984001 88.320799) (end 62.984001 89.542999) (width 0.25) (layer F.Cu) (net 31))
   (segment (start 68.539504 90.678018) (end 69.754001 89.463521) (width 0.25) (layer B.Cu) (net 31))
   (via (at 63.808237 58.547156) (size 0.8) (drill 0.4) (layers F.Cu B.Cu) (net 32))
