File: lopill.kicad/lopill.sch (KiCad schematic (older format))
At the start: 32 parts, among them J1 Pins Left, J2 SWD, J3 USB_B_Micro, J4 Pins Right, SW1 Reset, U1 XC6206PxxxMR, U2 STM32L052C8Tx, Y1 8MHz, Y2 32.768KHz

Commit message: Add 3D model of 8MHz crystal
Parts:
- Y1: footprint Crystal:Crystal_SMD_5032-2Pin_5.0x3.2mm -> lopill:Crystal_SMD_5032-2Pin_5.0x3.2mm_YXC
Changed lines of the file:
@@
 F 0 "Y1" V 5954 1481 50  0000 L CNN
 F 1 "8MHz" V 6045 1481 50  0000 L CNN
-F 2 "Crystal:Crystal_SMD_5032-2Pin_5.0x3.2mm" H 6000 1350 50  0001 C CNN
+F 2 "lopill:Crystal_SMD_5032-2Pin_5.0x3.2mm_YXC" H 6000 1350 50  0001 C CNN
 F 3 "https://datasheet.lcsc.com/szlcsc/1903061615_Yangxing-Tech-X50328MSB2GI_C115962.pdf" H 6000 1350 50  0001 C CNN
 F 4 "C115962" H 6000 1350 50  0001 C CNN "LCSC"

Commit message: Disconnect USB shield from ground
Parts:
- J3: symbol Connector:USB_B_Micro -> lopill-rescue:USB_B_Micro-Connector
Connections:
- net GND: no longer J3.6 (Shield)
- no-connect marks 1 -> 2
Changed lines of the file:
@@
 L power:GND #PWR0109
 U 1 1 5F02FFC2
-P 2550 5500
-F 0 "#PWR0109" H 2550 5250 50  0001 C CNN
-F 1 "GND" H 2555 5327 50  0000 C CNN
-F 2 "" H 2550 5500 50  0001 C CNN
-F 3 "" H 2550 5500 50  0001 C CNN
-	1    2550 5500
+P 2600 5500
+F 0 "#PWR0109" H 2600 5250 50  0001 C CNN
+F 1 "GND" H 2605 5327 50  0000 C CNN
+F 2 "" H 2600 5500 50  0001 C CNN
+F 3 "" H 2600 5500 50  0001 C CNN
+	1    2600 5500
 	1    0    0    -1
 $EndComp
-Wire Wire Line
-	2500 5500 2550 5500
-Connection ~ 2550 5500
-Wire Wire Line
-	2550 5500 2600 5500
 $Comp
 L power:GND #PWR0110
@@
 $EndComp
 $Comp
-L Connector:USB_B_Micro J3
-U 1 1 5F02DD0A
-P 2600 5100
-F 0 "J3" H 2657 5567 50  0000 C CNN
-F 1 "USB_B_Micro" H 2657 5476 50  0000 C CNN
-F 2 "lopill:USB_Micro-B_HRO_U-D-M5DD-W-1_Vertical" H 2750 5050 50  0001 C CNN
-F 3 "https://datasheet.lcsc.com/szlcsc/1811151141_Korean-Hroparts-Elec-U-D-M5DD-W-1_C145795.pdf" H 2750 5050 50  0001 C CNN
-F 4 "C145795" H 2600 5100 50  0001 C CNN "LCSC"
-F 5 "Korean Hroparts Elec U-D-M5DD-W-1" H 2600 5100 50  0001 C CNN "Product"
-	1    2600 5100
-	1    0    0    -1
-$EndComp
-$Comp
 L Device:Crystal Y2
 U 1 1 5F02594C
@@
 Text Label 8200 2450 0    50   ~ 0
 PC13
+$Comp
+L lopill-rescue:USB_B_Micro-Connector J3
+U 1 1 5F02DD0A
+P 2600 5100
+F 0 "J3" H 2657 5567 50  0000 C CNN
+F 1 "USB_B_Micro" H 2657 5476 50  0000 C CNN
+F 2 "lopill:USB_Micro-B_HRO_U-D-M5DD-W-1_Vertical" H 2750 5050 50  0001 C CNN
+F 3 "https://datasheet.lcsc.com/szlcsc/1811151141_Korean-Hroparts-Elec-U-D-M5DD-W-1_C145795.pdf" H 2750 5050 50  0001 C CNN
+F 4 "C145795" H 2600 5100 50  0001 C CNN "LCSC"
+F 5 "Korean Hroparts Elec U-D-M5DD-W-1" H 2600 5100 50  0001 C CNN "Product"
+	1    2600 5100
+	1    0    0    -1
+$EndComp
+NoConn ~ 2500 5500
 $EndSCHEMATC
