File: lopill.kicad/lopill.kicad_sch (KiCad schematic)
At the start: 32 parts, among them J1 Pins Left, J2 SWD, J3 USB_B_Micro, J4 Pins Right, SW1 Reset, U1 XC6206PxxxMR, U2 STM32L052C8Tx, Y1 8MHz, Y2 32.768KHz

Commit message: Move footprints to the shared library
Parts:
- SW1: footprint lopill:SW_Push_1P1T_NO_5.1x5.1mm_H2.5mm -> spbnick:SW_Push_1P1T_NO_5.1x5.1mm_H2.5mm
- Y1: footprint lopill:Crystal_SMD_5032-2Pin_5.0x3.2mm_YXC -> spbnick:Crystal_SMD_5032-2Pin_5.0x3.2mm_YXC
Changed lines of the file:
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@@
       (effects (font (size 1.27 1.27)) (justify left))
     )
-    (property "Footprint" "lopill:Crystal_SMD_5032-2Pin_5.0x3.2mm_YXC" (id 2) (at 152.4 34.29 0)
+    (property "Footprint" "spbnick:Crystal_SMD_5032-2Pin_5.0x3.2mm_YXC" (id 2) (at 152.4 34.29 0)
       (effects (font (size 1.27 1.27)) hide)
     )
@@
     (property "Reference" "SW1" (id 0) (at 144.78 77.851 0))
     (property "Value" "Reset" (id 1) (at 144.78 80.1624 0))
-    (property "Footprint" "lopill:SW_Push_1P1T_NO_5.1x5.1mm_H2.5mm" (id 2) (at 144.78 80.01 0)
+    (property "Footprint" "spbnick:SW_Push_1P1T_NO_5.1x5.1mm_H2.5mm" (id 2) (at 144.78 80.01 0)
       (effects (font (size 1.27 1.27)) hide)
     )
@@
     )
     (path "/00000000-0000-0000-0000-00005f927b2e"
-      (reference "SW1") (unit 1) (value "Reset") (footprint "lopill:SW_Push_1P1T_NO_5.1x5.1mm_H2.5mm")
+      (reference "SW1") (unit 1) (value "Reset") (footprint "spbnick:SW_Push_1P1T_NO_5.1x5.1mm_H2.5mm")
     )
     (path "/00000000-0000-0000-0000-00005f01e784"
@@
     )
     (path "/00000000-0000-0000-0000-00005f03b734"
-      (reference "Y1") (unit 1) (value "8MHz") (footprint "lopill:Crystal_SMD_5032-2Pin_5.0x3.2mm_YXC")
+      (reference "Y1") (unit 1) (value "8MHz") (footprint "spbnick:Crystal_SMD_5032-2Pin_5.0x3.2mm_YXC")
     )
     (path "/00000000-0000-0000-0000-00005f02594c"
